File: kicad/power_supply/power_supply.kicad_pcb (KiCad board)
At the start: 2 copper layers, 110.5 x 48 mm, 18 parts, among them J1 AC IN, J2 DC OUT

Commit message: Production candidate
Parts:
- removed R1, R2: 1k, Resistor_THT:R_Axial_DIN0414_L11.9mm_D4.5mm_P15.24mm_Horizontal
- added J3: CT, Custom:Spade Connector, F.Cu at (163.3, 80.8)
- added J3: CT, Custom:Spade Connector, F.Cu at (151.4, 80.8)
- added J4: AC2, Custom:Spade Connector, F.Cu at (71.4, 69.2)
- added J5: V-, Custom:Spade Connector, F.Cu at (151.4, 90.9)
- added J5: V-, Custom:Spade Connector, F.Cu at (163.3, 90.9)
- added J6: V+, Custom:Spade Connector, F.Cu at (151.4, 71.1)
- added J6: V+, Custom:Spade Connector, F.Cu at (163.3, 71.1)
- J1: value AC IN -> AC1; footprint TerminalBlock_Phoenix:TerminalBlock_Phoenix_PT-1,5-3-3.5-H_1x03_P3.50mm_Horizontal -> Custom:Spade Connector
- J2: value DC OUT -> GND; footprint TerminalBlock_Phoenix:TerminalBlock_Phoenix_PT-1,5-3-3.5-H_1x03_P3.50mm_Horizontal -> Custom:Spade Connector
- moved J2 89.4 mm to (71.4, 80.4), turned to 0 degrees
- moved J1 13.1 mm to (71.6, 92.0), turned to 0 degrees
- moved D1 8.89 mm to (97.8, 69.8)
- moved D2 8.89 mm to (83.1, 90.2)
- moved D3 8.89 mm to (83.1, 69.8)
- moved D4 8.89 mm to (97.8, 90.2)
- moved REF** 7.87 mm to (68.8, 66.3)
- moved REF** 7.87 mm to (68.8, 104.6)
- moved REF** 4.89 mm to (165.6, 66.0)
- moved REF** 4.89 mm to (165.6, 104.7)
Connections:
- J1 pad 1: /AC2 -> /AC1
- J1 pad 2: GND -> /AC1
- J2 pad 1: /V- -> GND
Routing:
- net /AC2: track 19.7 -> 25.3 mm
- net /V-: track 92.4 -> 93.7 mm
- net /V+: track 94.7 -> 94.2 mm
Other:
- board size 110.5 x 48 mm -> 105.7 x 48 mm
- board text added: "Designed by Pontus Rydin. https://github.com/prydin/classab-amp-mosfet"
- board text removed: "CT"
- board text removed: "Designed by Pontus Rydin. https://github.com/prydin/classab-amp"

Commit message: Public release candidate
Parts:
- added C7: 100n, Capacitor_THT:C_Rect_L7.2mm_W5.5mm_P5.00mm_FKS2_FKP2_MKS2_MKP2, F.Cu at (74.4, 106.6)
- added R3: 220, Resistor_THT:R_Axial_DIN0414_L11.9mm_D4.5mm_P7.62mm_Vertical, F.Cu at (66.8, 97.0)
- moved J1 8.17 mm to (69.8, 84.1)
- moved J2 4.10 mm to (69.8, 76.6)
- moved J4 1.52 mm to (69.8, 69.2)
- moved REF** 1.52 mm to (67.3, 66.3)
- moved REF** 1.52 mm to (67.3, 104.6)
Connections:
- REF** pad 1: GND -> GNDPWR
Routing:
- net GNDPWR: track 0.00 -> 13.0 mm
- net /AC1: track 39.2 -> 44.4 mm
Other:
- board size 105.7 x 48 mm -> 106.9 x 48 mm

Commit message: Adjusted power supply
Parts:
- removed C7: 100n, Capacitor_THT:C_Rect_L7.2mm_W5.5mm_P5.00mm_FKS2_FKP2_MKS2_MKP2
- removed R3: 220, Resistor_THT:R_Axial_DIN0414_L11.9mm_D4.5mm_P7.62mm_Vertical
Connections:
- REF** pad 1: GNDPWR -> GND
Routing:
- net GNDPWR: track 13.0 -> 0.00 mm
