File: kicad/power_supply/power_supply.kicad_sch (KiCad schematic)
At the start: 14 parts, among them J1 AC IN, J2 DC OUT

Commit message: Production candidate
Parts:
- removed J1: AC IN, TerminalBlock_Phoenix:TerminalBlock_Phoenix_PT-1,5-3-3.5-H_1x03_P3.50mm_Horizontal, symbol Connector:Screw_Terminal_01x03
- removed J2: DC OUT, TerminalBlock_Phoenix:TerminalBlock_Phoenix_PT-1,5-3-3.5-H_1x03_P3.50mm_Horizontal, symbol Connector:Screw_Terminal_01x03
- added J1: AC1, Custom:Spade Connector, symbol CustomSymbols:Spade_Connector
- added J2: GND, Custom:Spade Connector, symbol CustomSymbols:Spade_Connector
- added J3: CT, Custom:Spade Connector, symbol CustomSymbols:Spade_Connector
- added J4: AC2, Custom:Spade Connector, symbol CustomSymbols:Spade_Connector
- added J5: V-, Custom:Spade Connector, symbol CustomSymbols:Spade_Connector
- added J6: V+, Custom:Spade Connector, symbol CustomSymbols:Spade_Connector
Connections:
- net AC1: now also J1.1, J1.2
- net AC2: now also J4.1, J4.2
- net GND: now also J2.1, J2.2, J3.1, J3.2
- net V+: now also J6.1, J6.2
- net V-: now also J5.1, J5.2

Commit message: Public release candidate
Parts:
- removed R1, R2: 1k, Resistor_THT:R_Axial_DIN0414_L11.9mm_D4.5mm_P15.24mm_Horizontal, symbol Device:R
- added C7: 100n, Capacitor_THT:C_Rect_L7.2mm_W5.5mm_P5.00mm_FKS2_FKP2_MKS2_MKP2, symbol Device:C
- added R3: 220, Resistor_THT:R_Axial_DIN0414_L11.9mm_D4.5mm_P7.62mm_Vertical, symbol Device:R
Connections:
- net GND: now also C7.1, R3.1
- new net GNDPWR: C7.2, R3.2
Other:
- note added: "3W"
- note removed: "5W"
- moved on the sheet: J2, J5, J6

Commit message: Adjusted power supply
Parts:
- removed C7: 100n, Capacitor_THT:C_Rect_L7.2mm_W5.5mm_P5.00mm_FKS2_FKP2_MKS2_MKP2, symbol Device:C
- removed R3: 220, Resistor_THT:R_Axial_DIN0414_L11.9mm_D4.5mm_P7.62mm_Vertical, symbol Device:R
Other:
- note removed: "3W"
