File: kicad/classab-amp.kicad_sch (KiCad schematic)
At the start: 68 parts, among them J1 SPEAKER, J3 INPUT, Q1 BC547, Q10 MJL3281C, Q11 BD140, Q12 MJL1302C, Q13 BC547, Q14 BC557, Q2 BC547, Q3 BC557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

Commit message: Production candidate
Parts:
- removed C1: 33u, Capacitor_THT:CP_Radial_D4.0mm_P1.50mm, symbol Device:C_Polarized
- removed C11, C12: 470p, Capacitor_THT:C_Rect_L7.2mm_W3.0mm_P5.00mm_FKS2_FKP2_MKS2_MKP2, symbol Device:C
- removed C8: 4.7n, Capacitor_THT:C_Rect_L7.2mm_W3.0mm_P5.00mm_FKS2_FKP2_MKS2_MKP2, symbol Device:C
- removed D1, D2: 1N4148, Diode_THT:D_DO-35_SOD27_P7.62mm_Horizontal, symbol Diode:1N4148
- removed D3, D6: 1N4004, Diode_THT:D_DO-41_SOD81_P10.16mm_Horizontal, symbol Diode:1N4004
- removed Q1, Q13, Q2, Q5: BC547, Package_TO_SOT_THT:TO-92_Inline, symbol Transistor_BJT:BC547
- removed Q10: MJL3281C, Package_TO_SOT_THT:TO-264-3_Vertical, symbol Custom:MJL3218C
- removed Q11: BD140, Package_TO_SOT_THT:TO-126-3_Vertical, symbol Transistor_BJT:BD140
- removed Q12: MJL1302C, Package_TO_SOT_THT:TO-264-3_Vertical, symbol Custom:MJL1302C
- removed Q14, Q3, Q4: BC557, Package_TO_SOT_THT:TO-92_Inline, symbol Transistor_BJT:BC557
- removed Q9: BD139, Package_TO_SOT_THT:TO-126-3_Vertical, symbol Transistor_BJT:BD139
- removed R22, R23: 150, Resistor_THT:R_Axial_DIN0204_L3.6mm_D1.6mm_P7.62mm_Horizontal, symbol Device:R
- removed R24, R27: 1k, Resistor_THT:R_Axial_DIN0204_L3.6mm_D1.6mm_P7.62mm_Horizontal, symbol Device:R
- removed R25, R26: 8.2k, Resistor_THT:R_Axial_DIN0204_L3.6mm_D1.6mm_P7.62mm_Horizontal, symbol Device:R
- added C1: 33u, Capacitor_THT:CP_Radial_D4.0mm_P2.00mm, symbol Device:C
- added D11, D6: 1N5919, Diode_THT:D_DO-41_SOD81_P10.16mm_Horizontal, symbol Device:D_Zener
- added J2, J4, J5: ~, footprints:Spade Connector, symbol Custom:Spade_Connector
- added Q1, Q11, Q12, Q15, Q2: 2N5551, Package_TO_SOT_THT:TO-92_Wide, symbol Custom:2N5551
- added Q10: IRFP9240, Package_TO_SOT_THT:TO-247-3_Vertical, symbol Custom:IRFP9240
- added Q16, Q3, Q4: 2N5401, Package_TO_SOT_THT:TO-92_Wide, symbol Custom:2N5401
- added Q9: IRFP240, Package_TO_SOT_THT:TO-247-3_Vertical, symbol Custom:IRFP240
- added R8: 330, Resistor_THT:R_Axial_DIN0204_L3.6mm_D1.6mm_P7.62mm_Horizontal, symbol Device:R
- added RV2: 300, footprints:TRIM_T93YA103KT20, symbol Device:R_Potentiometer_Trim
- C2: value 220p -> 100p
- C5: value 50p -> 100p
- C6: value 100n -> 10u; footprint Capacitor_THT:C_Rect_L7.2mm_W3.0mm_P5.00mm_FKS2_FKP2_MKS2_MKP2 -> Capacitor_THT:CP_Radial_D4.0mm_P2.00mm
- R1, R2: footprint Resistor_THT:R_Axial_DIN0204_L3.6mm_D1.6mm_P7.62mm_Horizontal -> Resistor_THT:R_Axial_DIN0207_L6.3mm_D2.5mm_P2.54mm_Vertical
- R10, R14: value 150 -> 100
- R11: value 22k -> 4.7k; footprint Resistor_THT:R_Axial_DIN0204_L3.6mm_D1.6mm_P7.62mm_Horizontal -> Resistor_THT:R_Axial_DIN0207_L6.3mm_D2.5mm_P2.54mm_Vertical
- R12: value 15k -> 330; footprint Resistor_THT:R_Axial_DIN0204_L3.6mm_D1.6mm_P7.62mm_Horizontal -> Resistor_THT:R_Axial_DIN0207_L6.3mm_D2.5mm_P2.54mm_Vertical
- R16, R17: value 0.22 -> 0.33
- R18: value 1.5k -> 330
- R19: value 1.5k -> 1k
- R20: footprint Resistor_THT:R_Axial_DIN0414_L11.9mm_D4.5mm_P15.24mm_Horizontal -> Resistor_THT:R_Axial_DIN0516_L15.5mm_D5.0mm_P5.08mm_Vertical
- R3, R4, R5: value 1k -> 470
- R6: value 10k -> 4.7k
- R7: value 1k -> 2.2k
- R9: value 22k -> 47k
- RV1: value 10k -> 300
Connections:
- net B+: now also R19.1, J4.1, J4.2, Q9.2 (D)
- net B-: now also J2.1, J2.2, Q10.2 (D), Q11.1 (E), Q12.1 (E); no longer D5.1 (K)
- net GND: now also R2.1, Q16.3 (C); no longer C13.1, C14.2, C15.2, C16.1, D10.1 (K), D7.2 (A), J1.2 (Pin_2), R2.2, R20.2
- net LTP COM: now also Q1.3 (C), Q3.2 (B), Q3.3 (C), Q4.2 (B)
- net at C6.2, Q7.1 (E), Q8.2 (C)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: now also D4.1 (K), R18.1
- net at D8.2 (A), R16.1: now also Q9.3 (S); no longer R18.2
- net at C3.1, L1.1, R16.2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: now also D5.1 (K), D11.1 (K)
- net at C5.2, C6.1, Q6.2 (C)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: now also D6.1 (K), R8.1
- net at C5.1: now also Q16.2 (B), Q2.3 (C), Q4.3 (C); no longer Q6.3 (B)
- net at D9.1 (K), R17.2: now also Q10.3 (S); no longer R19.1
- net at D5.2 (A): now also D6.2 (A); no longer D4.1 (K)
- net at Q8.3 (B), R13.1: now also Q12.3 (C); no longer D4.2 (A)
- net at R19.2: now also Q6.3 (B), Q16.1 (E)
- net at C2.1, R1.2: now also R2.2, Q2.2 (B); no longer R2.1
- net at R3.2: now also Q4.1 (E)
- net at R6.1: now also Q11.3 (C), Q15.2 (B)
- net at Q8.1 (E), R14.1: now also Q12.2 (B)
- net at C4.1, R9.1: now also Q1.2 (B)
- net at R5.1: now also Q11.2 (B), Q15.1 (E)
- net at R4.2: now also Q3.1 (E)
- net at C3.2: now also R20.2; no longer R20.1
- net at R1.1: now also C1.2
- net INPUT: no longer names the net of J3.2 (Pin_2)
- net INPUT: now also C1.1
- new net: Q1.1 (E), RV2.1
- new net: Q15.3 (C), RV2.2
- new net: Q2.1 (E), RV2.3
- new net: Q9.1 (G), R8.2
- new net: D11.2 (A), D4.2 (A)
- new net: Q10.1 (G), R18.2
- new net PWRGND: C13.1, C14.2, C15.2, C16.1, D10.1 (K), D7.2 (A), J1.2 (Pin_2), J5.1, J5.2, R20.1
Other:
- note added: "Non-polarized"
- note added: "Trim for 0V output offset"
- note removed: "C8 optional. Omit if amp is stable without it."
- note removed: "R22 and R23 should be closely matched."
- moved on the sheet: C13, C14, C15, C16, C2, C3, C4, C5, C6, C7, D10, D7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

Commit message: Production candidate
Parts:
- R1: value 2.2k -> 150
- R7: value 2.2k -> 1k
- R9: value 47k -> 22k
Changed lines of the file:
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@@
 			)
 		)
-		(property "Value" "47k"
+		(property "Value" "22k"
 			(at 118.11 80.01 90)
 			(effects
@@
 			)
 		)
-		(property "Value" "2.2k"
+		(property "Value" "1k"
 			(at 110.49 100.3299 0)
 			(effects
@@
 			)
 		)
-		(property "Value" "2.2k"
+		(property "Value" "150"
 			(at 44.45 80.01 90)
 			(effects

Commit message: Public release candidate
Connections:
- no-connect marks 0 -> 1
Changed lines of the file:
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@@
 		(color 0 0 0 0)
+	)
+	(no_connect
+		(at 116.84 101.6)
 	)
 	(wire

Commit message: Adjusted power supply
Parts:
- added R22: 100, Resistor_THT:R_Axial_DIN0204_L3.6mm_D1.6mm_P7.62mm_Horizontal, symbol Device:R
Connections:
- net PWRGND: now also C2.2, C7.1, Q16.3 (C), R13.2, R15.2, R2.1, R6.2, R7.1, R22.2
- removed net GND: C2.2, C7.1, J3.1 (Pin_1), Q16.3 (C), R13.2, R15.2, R2.1, R6.2, R7.1
- new net GNDS: J3.1 (Pin_1), R22.1
Other:
- moved on the sheet: J3
Changed lines of the file:
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@@
 	)
 	(junction
+		(at 39.37 99.06)
+		(diameter 0)
+		(color 0 0 0 0)
+	)
+	(junction
+		(at 33.02 86.36)
+		(diameter 0)
+		(color 0 0 0 0)
+	)
+	(junction
 		(at 62.23 83.82)
 		(diameter 0)
@@
 	)
 	(junction
-		(at 29.21 83.82)
-		(diameter 0)
-		(color 0 0 0 0)
-	)
-	(junction
 		(at 163.83 143.51)
 		(diameter 0)
@@
 	(wire
 		(pts
-			(xy 25.4 83.82) (xy 29.21 83.82)
-		)
-		(stroke
-			(width 0)
-			(type default)
-		)
-	)
-	(wire
-		(pts
 			(xy 39.37 114.3) (xy 39.37 115.57)
 		)
@@
 	(wire
 		(pts
+			(xy 39.37 88.9) (xy 39.37 86.36)
+		)
+		(stroke
+			(width 0)
+			(type default)
+		)
+	)
+	(wire
+		(pts
 			(xy 179.07 130.81) (xy 180.34 130.81)
 		)
@@
 	(wire
 		(pts
-			(xy 29.21 86.36) (xy 33.02 86.36)
+			(xy 25.4 86.36) (xy 33.02 86.36)
 		)
 		(stroke
@@
 	(wire
 		(pts
-			(xy 25.4 82.55) (xy 25.4 83.82)
+			(xy 82.55 130.81) (xy 82.55 127)
 		)
 		(stroke
@@
 	(wire
 		(pts
-			(xy 82.55 130.81) (xy 82.55 127)
+			(xy 92.71 41.91) (xy 92.71 45.72)
 		)
 		(stroke
@@
 	(wire
 		(pts
-			(xy 92.71 41.91) (xy 92.71 45.72)
+			(xy 142.24 143.51) (xy 128.27 143.51)
 		)
 		(stroke
@@
 	(wire
 		(pts
-			(xy 142.24 143.51) (xy 128.27 143.51)
+			(xy 142.24 31.75) (xy 128.27 31.75)
 		)
 		(stroke
@@
 	(wire
 		(pts
-			(xy 142.24 31.75) (xy 128.27 31.75)
+			(xy 25.4 83.82) (xy 33.02 83.82)
 		)
 		(stroke
@@
 	(wire
 		(pts
+			(xy 33.02 86.36) (xy 39.37 86.36)
+		)
+		(stroke
+			(width 0)
+			(type default)
+		)
+	)
+	(wire
+		(pts
 			(xy 39.37 114.3) (xy 50.8 114.3)
 		)
@@
 	(wire
 		(pts
+			(xy 39.37 96.52) (xy 39.37 99.06)
+		)
+		(stroke
+			(width 0)
+			(type default)
+		)
+	)
+	(wire
+		(pts
 			(xy 187.96 93.98) (xy 187.96 97.79)
 		)
@@
 	(wire
 		(pts
-			(xy 29.21 83.82) (xy 33.02 83.82)
-		)
-		(stroke
-			(width 0)
-			(type default)
-		)
-	)
-	(wire
-		(pts
 			(xy 176.53 22.86) (xy 187.96 22.86)
 		)
@@
 				)
 				(justify left)
+				(hide yes)
 			)
 		)
@@
 	)
 	(symbol
+		(lib_id "Device:R")
+		(at 39.37 92.71 0)
+		(unit 1)
+		(exclude_from_sim no)
+		(in_bom yes)
+		(on_board yes)
+		(dnp no)
+		(fields_autoplaced yes)
+		(property "Reference" "R22"
+			(at 41.91 91.4399 0)
+			(effects
+				(font
+					(size 1.27 1.27)
+				)
+				(justify left)
+			)
+		)
+		(property "Value" "100"
+			(at 41.91 93.9799 0)
+			(effects
+				(font
+					(size 1.27 1.27)
+				)
+				(justify left)
+			)
+		)
+		(property "Footprint" "Resistor_THT:R_Axial_DIN0204_L3.6mm_D1.6mm_P7.62mm_Horizontal"
+			(at 37.592 92.71 90)
+			(effects
+				(font
+					(size 1.27 1.27)
+				)
+				(hide yes)
+			)
+		)
+		(property "Datasheet" "~"
+			(at 39.37 92.71 0)
+			(effects
+				(font
+					(size 1.27 1.27)
+				)
+				(hide yes)
+			)
+		)
+		(property "Description" "Resistor"
+			(at 39.37 92.71 0)
+			(effects
+				(font
+					(size 1.27 1.27)
+				)
+				(hide yes)
+			)
+		)
+		(pin "2"
+		)
+		(pin "1"
+		)
+		(instances
+			(project ""
+				(path "/856f1e14-388c-4d87-abe9-3c0c6310ec29"
+					(reference "R22")
+					(unit 1)
+				)
+			)
+		)
+	)
+	(symbol
 		(lib_id "Transistor_BJT:BD140")
 		(at 139.7 46.99 0)
@@
 		(on_board yes)
 		(dnp no)
-		(fields_autoplaced yes)
 		(property "Reference" "#PWR08"
 			(at 128.27 64.77 0)
@@
 			)
 		)
-		(property "Value" "GND"
-			(at 128.27 63.5 0)
+		(property "Value" "PWRGND"
+			(at 125.984 62.738 0)
 			(effects
 				(font
@@
 	(symbol
 		(lib_id "Connector:Screw_Terminal_01x02")
-		(at 24.13 86.36 180)
+		(at 20.32 86.36 180)
 		(unit 1)
 		(exclude_from_sim no)
@@
 		(fields_autoplaced yes)
 		(property "Reference" "J3"
-			(at 24.13 77.47 0)
+			(at 20.32 77.47 0)
 			(effects
 				(font
@@
 		)
 		(property "Value" "INPUT"
-			(at 24.13 80.01 0)
+			(at 20.32 80.01 0)
 			(effects
 				(font
@@
 		)
 		(property "Footprint" "TerminalBlock_4Ucon:TerminalBlock_4Ucon_1x02_P3.50mm_Horizontal"
-			(at 24.13 86.36 0)
+			(at 20.32 86.36 0)
 			(effects
 				(font
@@
 		)
 		(property "Datasheet" "~"
-			(at 24.13 86.36 0)
+			(at 20.32 86.36 0)
 			(effects
 				(font
@@
 		)
 		(property "Description" ""
-			(at 24.13 86.36 0)
+			(at 20.32 86.36 0)
 			(effects
 				(font
@@
 			)
 		)
-		(property "Value" "GND"
+		(property "Value" "PWRGND"
 			(at 62.23 107.95 0)
 			(effects
@@
 			)
 		)
-		(property "Value" "GND"
+		(property "Value" "PWRGND"
 			(at 115.57 142.24 0)
 			(effects
@@
 			)
 		)
-		(property "Value" "GND"
+		(property "Value" "PWRGND"
 			(at 50.8 137.16 0)
 			(effects
@@
 			)
 		)
-		(property "Value" "GND"
+		(property "Value" "GNDS"
 			(at 33.02 97.79 0)
 			(effects
@@
 			)
 		)
-		(property "Value" "GND"
+		(property "Value" "PWRGND"
 			(at 107.95 110.49 0)
 			(effects

Commit message: Minor changes
Other:
- note added: "-24V - -40V"
- note added: "24V - 40V"
Changed lines of the file:
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@@
 	(text "Wrap 16-18 AWG wire 10-12 turns around R21"
 		(exclude_from_sim no)
-		(at 224.028 71.12 0)
+		(at 244.348 73.914 0)
 		(effects
 			(font
@@
 		(effects
 			(font
+				(size 1.27 1.27)
+			)
+		)
+	)
+	(text "-24V - -40V"
+		(exclude_from_sim no)
+		(at 216.154 143.764 0)
+		(effects
+			(font
+				(size 1.27 1.27)
+			)
+		)
+	)
+	(text "24V - 40V"
+		(exclude_from_sim no)
+		(at 216.662 32.004 0)
+		(effects
+			(font

Commit message: Added protection diode for VAS. Removed offset pot.
Parts:
- removed RV2: 300, footprints:TRIM_T93YA103KT20, symbol Device:R_Potentiometer_Trim
- added D1: 1N4148, Diode_THT:D_DO-35_SOD27_P7.62mm_Horizontal, symbol Diode:1N4148
- added R23, R24: 100, Resistor_THT:R_Axial_DIN0207_L6.3mm_D2.5mm_P2.54mm_Vertical, symbol Device:R
- C1: value 33u -> 4.7u
- L1: value 10u -> 3u
Connections:
- net at C5.1, Q16.2 (B), Q2.3 (C)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: now also D1.1 (K)
- net at C5.2, C6.1, D6.1 (K)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: now also D1.2 (A)
- net at Q1.1 (E): now also R23.2
- net at Q15.3 (C): now also R23.1, R24.2
- net at Q2.1 (E): now also R24.1
Other:
- note removed: "Trim for 0V output offset"

Commit message: 2.0 stuff
Parts:
- removed C6: 10u, Capacitor_THT:CP_Radial_D4.0mm_P2.00mm, symbol Device:C
- removed D1, D5: 1N4148, Diode_THT:D_DO-35_SOD27_P7.62mm_Horizontal, symbol Diode:1N4148
- removed D11, D6: 1N5919, Diode_THT:D_DO-41_SOD81_P10.16mm_Horizontal, symbol Device:D_Zener
- removed D8, D9: 1N4004, Diode_THT:D_DO-41_SOD81_P10.16mm_Horizontal, symbol Diode:1N4004
- removed Q1, Q2: 2N5551, Package_TO_SOT_THT:TO-92_Wide, symbol Custom:2N5551
- removed Q6: BD140, Package_TO_SOT_THT:TO-126-3_Vertical, symbol Transistor_BJT:BD140
- removed Q8: BD139, Package_TO_SOT_THT:TO-126-3_Vertical, symbol Transistor_BJT:BD139
- added C10, C9: 68p, Capacitor_THT:CP_Radial_D4.0mm_P2.00mm, symbol Device:C
- added C6: 10u, symbol Device:C_Polarized
- added C8: 220n, Capacitor_THT:CP_Radial_D4.0mm_P2.00mm, symbol Device:C
- added D1: BAV21, Diode_THT:D_DO-35_SOD27_P7.62mm_Horizontal, symbol Diode:BAV21
- added D2, D6: 1N4148, Diode_THT:D_DO-35_SOD27_P7.62mm_Horizontal, symbol Diode:1N4148
- added D3, D5: 1N5919, Diode_THT:D_DO-41_SOD81_P10.16mm_Horizontal, symbol Device:D_Zener
- added Q1, Q2, Q6: 2N5401, Package_TO_SOT_THT:TO-92_Wide, symbol Custom:2N5401
- added Q13: BD139, Package_TO_SOT_THT:TO-126-3_Vertical, symbol Transistor_BJT:BD139
- added Q14: BD140, Package_TO_SOT_THT:TO-126-3_Vertical, symbol Transistor_BJT:BD140
- added Q5, Q8: 2N5551, Package_TO_SOT_THT:TO-92_Wide, symbol Custom:2N5551
- added R25: 100, Resistor_THT:R_Axial_DIN0207_L6.3mm_D2.5mm_P2.54mm_Vertical, symbol Device:R
- C4: footprint Capacitor_THT:CP_Radial_D8.0mm_P5.00mm -> (none)
- R10: value 100 -> 47
- R11: value 4.7k -> 10k
- R12: value 330 -> 680
- R13: value 10k -> 1k
- R14: value 100 -> 10k; footprint Resistor_THT:R_Axial_DIN0204_L3.6mm_D1.6mm_P7.62mm_Horizontal -> Resistor_THT:R_Axial_DIN0207_L6.3mm_D2.5mm_P2.54mm_Vertical
- R18, R8: value 330 -> 47
- R19: value 1k -> 10k
- R23: value 100 -> 680
- R4: value 470 -> 1k
- R6: value 4.7k -> 22
Connections:
- net B+: now also Q4.1 (E), Q13.2 (C), Q6.1 (E); no longer R19.1, R3.1
- net B-: now also Q15.1 (E), R13.2, R3.2, R6.2, Q14.1 (E); no longer Q11.1 (E), Q12.1 (E), R14.2
- net LTP COM: now also Q2.1 (E), R25.2; no longer Q3.2 (B), Q3.3 (C), Q4.2 (B)
- net PWRGND: now also C4.2, Q12.3 (C), R14.2, R19.2, C10.2, C9.2, D2.2 (A); no longer Q16.3 (C), R13.2, R6.2, R7.1
- net at C3.1, L1.1, R16.2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: now also D4.1 (K), D5.1 (K)
- net at Q12.2 (B): now also C5.1, Q11.3 (C), Q15.3 (C), D1.2 (A), Q1.3 (C); no longer R14.1
- net at R13.1: now also Q12.1 (E), Q8.2 (B); no longer Q12.3 (C)
- net at Q15.2 (B), R6.1: now also Q8.1 (E); no longer Q11.3 (C)
- net at R10.2: now also Q16.1 (E), Q6.2 (B)
- net at Q7.2 (C), R11.1: now also Q16.3 (C), C6.1, C9.1, Q13.3 (B); no longer C5.2, R8.1
- net at R24.1: now also Q1.1 (E)
- net at Q9.1 (G), R8.2: now also D3.1 (K)
- net at C2.1, R1.2, R2.2: now also Q1.2 (B)
- net at R9.1: now also R7.2, Q2.2 (B); no longer C4.1
- net at D4.2 (A): now also D3.2 (A)
- net at Q10.1 (G), R18.2: now also D6.1 (K)
- net at Q7.1 (E), R12.2: now also C5.2, C10.1, C6.2, D1.1 (K), Q14.3 (B), Q8.3 (C); no longer D4.1 (K), R18.1
- net at R23.2: now also R18.1, C8.2, Q14.2 (C)
- net at Q3.1 (E), R4.2: now also Q4.2 (B)
- new net: Q3.2 (B), Q4.3 (C), R19.1
- new net: Q16.2 (B), Q6.3 (C), R14.1
- new net: D5.2 (A), D6.2 (A)
- new net: C8.1, Q13.1 (E), R23.1, R8.1
- new net: Q5.1 (E), R5.1
- new net: Q11.2 (B), Q2.3 (C), Q5.2 (B), Q5.3 (C)
- new net: C4.1, D2.1 (K), R7.1
- new net: Q11.1 (E), R3.1
- new net: Q3.3 (C), R24.2, R25.1
- no-connect marks 1 -> 0
Other:
- moved on the sheet: C1, C13, C14, C15, C16, C2, C3, C7, D10, D7, J1, J2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

Commit message: Pre re-layout
Parts:
- removed D1: BAV21, Diode_THT:D_DO-35_SOD27_P7.62mm_Horizontal, symbol Diode:BAV21
- removed J1: SPEAKER, TerminalBlock_Phoenix:TerminalBlock_Phoenix_MKDS-1,5-2_1x02_P5.00mm_Horizontal, symbol Connector:Screw_Terminal_01x02
- removed L1: 3u, Capacitor_THT:CP_Radial_D4.0mm_P1.50mm, symbol Device:L
- removed R16, R17: 0.33, Resistor_THT:R_Axial_DIN0414_L11.9mm_D4.5mm_P15.24mm_Horizontal, symbol Device:R
- removed R21: 10, Resistor_THT:R_Axial_DIN0414_L11.9mm_D4.5mm_P15.24mm_Horizontal, symbol Device:R
- added J1, J6: ~, footprints:Spade Connector, symbol Custom:Spade_Connector
- C10, C8, C9: footprint Capacitor_THT:CP_Radial_D4.0mm_P2.00mm -> Capacitor_THT:C_Rect_L7.2mm_W3.0mm_P5.00mm_FKS2_FKP2_MKS2_MKP2
- C4: footprint (none) -> Capacitor_THT:CP_Radial_D8.0mm_P5.00mm
- C5: value 100p -> 33p
- C6: footprint (none) -> Capacitor_THT:CP_Radial_D4.0mm_P2.00mm
- R1, R14, R2, R23: footprint Resistor_THT:R_Axial_DIN0207_L6.3mm_D2.5mm_P2.54mm_Vertical -> Resistor_THT:R_Axial_DIN0204_L3.6mm_D1.6mm_P7.62mm_Horizontal
- R20: footprint Resistor_THT:R_Axial_DIN0516_L15.5mm_D5.0mm_P5.08mm_Vertical -> Resistor_THT:R_Axial_DIN0414_L11.9mm_D4.5mm_P15.24mm_Horizontal
Connections:
- net B-: now also Q14.2 (C); no longer Q14.1 (E)
- net PWRGND: now also J6.1, J6.2
- net SPEAKER: now also C3.1, D4.1 (K), D5.1 (K), Q10.3 (S), Q9.3 (S), R9.2, J1.1, J1.2
- net at C8.2, R18.1, R23.2: now also Q14.1 (E); no longer Q14.2 (C)
Other:
- note removed: "Wrap 16-18 AWG wire 10-12 turns around R21"
- moved on the sheet: C3, J5, R20
