File: kicad/classab-amp.kicad_sch (KiCad schematic)
At the start: 66 parts, among them J3 INPUT, Q1 2N5401, Q10 IRFP9240, Q11 2N5551, Q12 2N5551, Q13 BD139, Q14 BD140, Q15 2N5551, Q16 2N5401, Q2 2N5401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

Commit message: WIP
Parts:
- removed Q16: 2N5401, Package_TO_SOT_THT:TO-92_Wide, symbol Custom:2N5401
- removed Q8: 2N5551, Package_TO_SOT_THT:TO-92_Wide, symbol Custom:2N5551
- added Q16: BD140, Package_TO_SOT_THT:TO-126-3_Vertical, symbol Transistor_BJT:BD140
- added Q8: BD139, Package_TO_SOT_THT:TO-126-3_Vertical, symbol Transistor_BJT:BD139
Connections:
- net at Q15.2 (B), R6.1: now also Q8.1 (E)
- net at Q6.3 (C), R14.1: now also Q16.3 (B)
- net at C6.1, C9.1, Q13.3 (B)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: now also Q16.2 (C)
- net at C10.1, C5.2, C6.2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: now also Q8.2 (C)
- net at Q12.1 (E), R13.1: now also Q8.3 (B)
- net at Q6.2 (B), R10.2: now also Q16.1 (E)
Changed lines of the file:
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@@
 	)
 	(junction
-		(at 142.24 135.89)
-		(diameter 0)
-		(color 0 0 0 0)
-	)
-	(junction
 		(at 82.55 113.03)
 		(diameter 0)
@@
 	)
 	(junction
+		(at 142.24 135.89)
+		(diameter 0)
+		(color 0 0 0 0)
+	)
+	(junction
 		(at 50.8 92.71)
 		(diameter 0)
@@
 	)
 	(symbol
+		(lib_id "Transistor_BJT:BD139")
+		(at 139.7 130.81 0)
+		(unit 1)
+		(exclude_from_sim no)
+		(in_bom yes)
+		(on_board yes)
+		(dnp no)
+		(property "Reference" "Q8"
+			(at 144.272 126.238 0)
+			(effects
+				(font
+					(size 1.27 1.27)
+				)
+				(justify left)
+			)
+		)
+		(property "Value" "BD139"
+			(at 144.272 128.778 0)
+			(effects
+				(font
+					(size 1.27 1.27)
+				)
+				(justify left)
+			)
+		)
+		(property "Footprint" "Package_TO_SOT_THT:TO-126-3_Vertical"
+			(at 144.78 132.715 0)
+			(effects
+				(font
+					(size 1.27 1.27)
+					(italic yes)
+				)
+				(justify left)
+				(hide yes)
+			)
+		)
+		(property "Datasheet" "http://www.st.com/internet/com/TECHNICAL_RESOURCES/TECHNICAL_LITERATURE/DATASHEET/CD00001225.pdf"
+			(at 139.7 130.81 0)
+			(effects
+				(font
+					(size 1.27 1.27)
+				)
+				(justify left)
+				(hide yes)
+			)
+		)
+		(property "Description" "1.5A Ic, 80V Vce, Low Voltage Transistor, TO-126"
+			(at 139.7 130.81 0)
+			(effects
+				(font
+					(size 1.27 1.27)
+				)
+				(hide yes)
+			)
+		)
+		(pin "1"
+		)
+		(pin "3"
+		)
+		(pin "2"
+		)
+		(instances
+			(project "classab-amp"
+				(path "/856f1e14-388c-4d87-abe9-3c0c6310ec29"
+					(reference "Q8")
+					(unit 1)
+				)
+			)
+		)
+	)
+	(symbol
 		(lib_id "power:GND")
 		(at 233.68 99.06 0)
@@
 	)
 	(symbol
-		(lib_id "power:PWR_FLAG")
-		(at 33.02 85.09 90)
+		(lib_id "Transistor_BJT:BD140")
+		(at 139.7 48.26 0)
+		(mirror x)
 		(unit 1)
 		(exclude_from_sim no)
@@
 		(on_board yes)
 		(dnp no)
-		(fields_autoplaced yes)
-		(property "Reference" "#FLG02"
-			(at 31.115 85.09 0)
+		(property "Reference" "Q16"
+			(at 144.78 49.5301 0)
 			(effects
 				(font
 					(size 1.27 1.27)
 				)
-				(hide yes)
+				(justify left)
 			)
 		)
-		(property "Value" "PWR_FLAG"
-			(at 29.21 85.0899 90)
+		(property "Value" "BD140"
+			(at 144.78 46.9901 0)
 			(effects
 				(font
@@
 			)
 		)
-		(property "Footprint" ""
-			(at 33.02 85.09 0)
+		(property "Footprint" "Package_TO_SOT_THT:TO-126-3_Vertical"
+			(at 144.78 46.355 0)
 			(effects
 				(font
 					(size 1.27 1.27)
+					(italic yes)
 				)
+				(justify left)
 				(hide yes)
 			)
 		)
-		(property "Datasheet" "~"
-			(at 33.02 85.09 0)
+		(property "Datasheet" "http://www.st.com/internet/com/TECHNICAL_RESOURCES/TECHNICAL_LITERATURE/DATASHEET/CD00001225.pdf"
+			(at 139.7 48.26 0)
 			(effects
 				(font
 					(size 1.27 1.27)
 				)
+				(justify left)
 				(hide yes)
 			)
 		)
-		(property "Description" "Special symbol for telling ERC where power comes from"
-			(at 33.02 85.09 0)
+		(property "Description" "1.5A Ic, 80V Vce, Low Voltage Transistor, TO-126"
+			(at 139.7 48.26 0)
 			(effects
 				(font
@@
 		(pin "1"
 		)
+		(pin "3"
+		)
+		(pin "2"
+		)
 		(instances
-			(project ""
+			(project "classab-amp"
 				(path "/856f1e14-388c-4d87-abe9-3c0c6310ec29"
-					(reference "#FLG02")
+					(reference "Q16")
 					(unit 1)
 				)
@@
 	)
 	(symbol
-		(lib_id "Custom:2N5551")
-		(at 139.7 130.81 0)
+		(lib_id "power:PWR_FLAG")
+		(at 33.02 85.09 90)
 		(unit 1)
 		(exclude_from_sim no)
@@
 		(on_board yes)
 		(dnp no)
-		(property "Reference" "Q8"
-			(at 144.78 129.5399 0)
+		(fields_autoplaced yes)
+		(property "Reference" "#FLG02"
+			(at 31.115 85.09 0)
 			(effects
 				(font
 					(size 1.27 1.27)
 				)
-				(justify left)
+				(hide yes)
 			)
 		)
-		(property "Value" "2N5551"
-			(at 144.78 132.0799 0)
+		(property "Value" "PWR_FLAG"
+			(at 29.21 85.0899 90)
 			(effects
 				(font
@@
 			)
 		)
-		(property "Footprint" "Package_TO_SOT_THT:TO-92_Wide"
-			(at 144.78 132.715 0)
+		(property "Footprint" ""
+			(at 33.02 85.09 0)
 			(effects
 				(font
 					(size 1.27 1.27)
-					(italic yes)
 				)
-				(justify left)
 				(hide yes)
 			)
 		)
-		(property "Datasheet" "https://www.onsemi.com/pub/Collateral/2N3903-D.PDF"
-			(at 139.7 130.81 0)
+		(property "Datasheet" "~"
+			(at 33.02 85.09 0)
 			(effects
 				(font
 					(size 1.27 1.27)
 				)
-				(justify left)
 				(hide yes)
 			)
 		)
-		(property "Description" "0.2A Ic, 40V Vce, Small Signal NPN Transistor, TO-92"
-			(at 139.7 130.81 0)
+		(property "Description" "Special symbol for telling ERC where power comes from"
+			(at 33.02 85.09 0)
 			(effects
 				(font
@@
 			)
 		)
-		(pin "3"
-		)
 		(pin "1"
 		)
-		(pin "2"
-		)
 		(instances
-			(project "classab-amp"
+			(project ""
 				(path "/856f1e14-388c-4d87-abe9-3c0c6310ec29"
-					(reference "Q8")
+					(reference "#FLG02")
 					(unit 1)
 				)
@@
 					(unit 1)
 				)
-			)
-		)
-	)
-	(symbol
-		(lib_id "Custom:2N5401")
-		(at 139.7 48.26 0)
-		(mirror x)
-		(unit 1)
-		(exclude_from_sim no)
-		(in_bom yes)
-		(on_board yes)
-		(dnp no)
-		(fields_autoplaced yes)
-		(property "Reference" "Q16"
-			(at 144.78 46.9899 0)
-			(effects
-				(font
-					(size 1.27 1.27)
-				)
-				(justify left)
-			)
-		)
-		(property "Value" "2N5401"
-			(at 144.78 49.5299 0)
-			(effects
-				(font
-					(size 1.27 1.27)
-				)
-				(justify left)
-			)
-		)
-		(property "Footprint" "Package_TO_SOT_THT:TO-92_Wide"
-			(at 144.78 46.355 0)
-			(effects
-				(font
-					(size 1.27 1.27)
-					(italic yes)
-				)
-				(justify left)
-				(hide yes)
-			)
-		)
-		(property "Datasheet" "https://www.onsemi.com/pub/Collateral/2N3906-D.PDF"
-			(at 139.7 48.26 0)
-			(effects
-				(font
-					(size 1.27 1.27)
-				)
-				(justify left)
-				(hide yes)
-			)
-		)
-		(property "Description" "-0.2A Ic, -40V Vce, Small Signal PNP Transistor, TO-92"
-			(at 139.7 48.26 0)
-			(effects
-				(font
-					(size 1.27 1.27)
-				)
-				(hide yes)
-			)
-		)
-		(pin "3"
-		)
-		(pin "1"
-		)
-		(pin "2"
-		)
-		(instances
-			(project ""
-				(path "/856f1e14-388c-4d87-abe9-3c0c6310ec29"
-					(reference "Q16")
-					(unit 1)
-				)

Commit message: WIP
Parts:
- removed C7: 10n, Capacitor_THT:C_Rect_L7.2mm_W3.0mm_P5.00mm_FKS2_FKP2_MKS2_MKP2, symbol Device:C
- added C11, C7: 4.7u, Capacitor_THT:CP_Radial_D4.0mm_P2.00mm, symbol Device:C_Polarized
- added D1: 1N4148, Diode_THT:D_DO-35_SOD27_P5.08mm_Vertical_KathodeUp, symbol Diode:1N4148
- added D8, D9: 1N4148, Diode_THT:D_DO-35_SOD27_P7.62mm_Horizontal, symbol Diode:1N4148
- added R16: 4.7k, Resistor_THT:R_Axial_DIN0204_L3.6mm_D1.6mm_P7.62mm_Horizontal, symbol Device:R
- R14, R19: value 10k -> 4.7k
- R15: value 220 -> 4.7k; footprint Resistor_THT:R_Axial_DIN0414_L11.9mm_D4.5mm_P15.24mm_Horizontal -> Resistor_THT:R_Axial_DIN0204_L3.6mm_D1.6mm_P7.62mm_Horizontal
- R20: footprint Resistor_THT:R_Axial_DIN0414_L11.9mm_D4.5mm_P15.24mm_Horizontal -> Resistor_THT:R_Axial_DIN0414_L11.9mm_D4.5mm_P5.08mm_Vertical
Connections:
- net B+: now also C11.1, C7.1
- net LTP COM: now also D1.1 (K)
- net PWRGND: now also R16.2; no longer R14.2, R19.2
- net at Q2.2 (B), R7.2, R9.1: now also D1.2 (A), D8.1 (K), D9.2 (A)
- net at C2.1, Q1.2 (B), R1.2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: now also D8.2 (A), D9.1 (K)
- net CHASSIS: no longer names the net of R15.1
- net CHASSIS: now also R19.2, C7.2
- new net: C11.2, R14.2, R16.1
Other:
- moved on the sheet: C2, R2
