File: kicad/classab-amp.kicad_pcb (KiCad board)
At the start: 2 copper layers, 87.4 x 101.9 mm, 75 parts, among them J1 SPEAKER, J3 INPUT, Q1 BC547, Q10 MJL3218C, Q11 BD140, Q12 MJL1302C, Q13 BC547, Q14 BC557, Q2 BC547, Q3 BC557, Q4 BC557, Q5 BC547, Q6 BD140, Q7 BD139, Q8 BD139, Q9 BD139

Commit message: Production candidate
Parts:
- removed the ? at (247.4, 119.4)
- removed the ? at (235.0, 103.1)
- removed the ? at (247.4, 43.2)
- removed the ? at (187.5, 129.5)
- removed C11, C12: 470p, Capacitor_THT:C_Rect_L7.2mm_W3.0mm_P5.00mm_FKS2_FKP2_MKS2_MKP2
- removed C8: 4.7n, Capacitor_THT:C_Rect_L7.2mm_W3.0mm_P5.00mm_FKS2_FKP2_MKS2_MKP2
- removed D1, D2: 1N4148, Diode_THT:D_DO-35_SOD27_P7.62mm_Horizontal
- removed D3: 1N4004, Diode_THT:D_DO-41_SOD81_P10.16mm_Horizontal
- removed PIC1: LOGO, LOGO
- removed Q13, Q5: BC547, Package_TO_SOT_THT:TO-92_Inline
- removed Q14: BC557, Package_TO_SOT_THT:TO-92_Inline
- removed R22, R23: 150, Resistor_THT:R_Axial_DIN0204_L3.6mm_D1.6mm_P7.62mm_Horizontal
- removed R24, R27: 1k, Resistor_THT:R_Axial_DIN0204_L3.6mm_D1.6mm_P7.62mm_Horizontal
- removed R25, R26: 8.2k, Resistor_THT:R_Axial_DIN0204_L3.6mm_D1.6mm_P7.62mm_Horizontal
- removed the REF** at (268.0, 35.0)
- removed the REF** at (267.0, 129.5)
- removed the REF** at (188.5, 35.0)
- added ?: , , F.Cu at (195.8, 109.2)
- added D11: 1N5919, Diode_THT:D_DO-41_SOD81_P10.16mm_Horizontal, F.Cu at (250.2, 87.6)
- added J2: ~, footprints:Spade Connector, F.Cu at (263.5, 104.8)
- added J4: ~, footprints:Spade Connector, F.Cu at (262.9, 30.5)
- added J5: ~, footprints:Spade Connector, F.Cu at (221.0, 85.7)
- added Q15: 2N5551, Package_TO_SOT_THT:TO-92_Wide, F.Cu at (203.8, 65.4)
- added Q16: 2N5401, Package_TO_SOT_THT:TO-92_Wide, F.Cu at (222.9, 59.2)
- added R8: 330, Resistor_THT:R_Axial_DIN0204_L3.6mm_D1.6mm_P7.62mm_Horizontal, F.Cu at (268.6, 67.3)
- added REF**: MountingHole_3.2mm_M3, MountingHole:MountingHole_3.2mm_M3, F.Cu at (273.7, 109.2)
- added REF**: MountingHole_3.2mm_M3, MountingHole:MountingHole_3.2mm_M3, F.Cu at (196.8, 34.3)
- added REF**: MountingHole_3.2mm_M3, MountingHole:MountingHole_3.2mm_M3, F.Cu at (273.7, 34.3)
- added RV2: 300, footprints:TRIM_T93YA103KT20, F.Cu at (211.5, 53.3)
- C2: value 220p -> 100p
- C5: value 50p -> 100p
- C6: value 100n -> 10u; footprint Capacitor_THT:C_Rect_L7.2mm_W3.0mm_P5.00mm_FKS2_FKP2_MKS2_MKP2 -> Capacitor_THT:CP_Radial_D4.0mm_P1.50mm
- D6: value 1N4004 -> 1N5919
- Q1, Q2: value BC547 -> 2N5551; footprint Package_TO_SOT_THT:TO-92_Inline -> Package_TO_SOT_THT:TO-92_Wide
- Q10: value MJL3218C -> IRFP9240; footprint Package_TO_SOT_THT:TO-264-3_Vertical -> Package_TO_SOT_THT:TO-247-3_Vertical
- Q11: value BD140 -> 2N5551; footprint Package_TO_SOT_THT:TO-126-3_Vertical -> Package_TO_SOT_THT:TO-92_Wide
- Q12: value MJL1302C -> 2N5551; footprint Package_TO_SOT_THT:TO-264-3_Vertical -> Package_TO_SOT_THT:TO-92_Wide
- Q3, Q4: value BC557 -> 2N5401; footprint Package_TO_SOT_THT:TO-92_Inline -> Package_TO_SOT_THT:TO-92_Wide
- Q9: value BD139 -> IRFP240; footprint Package_TO_SOT_THT:TO-126-3_Vertical -> Package_TO_SOT_THT:TO-247-3_Vertical
- R1, R2: footprint Resistor_THT:R_Axial_DIN0204_L3.6mm_D1.6mm_P7.62mm_Horizontal -> Resistor_THT:R_Axial_DIN0207_L6.3mm_D2.5mm_P2.54mm_Vertical
- R10, R14: value 150 -> 100
- R11: value 22k -> 4.7k; footprint Resistor_THT:R_Axial_DIN0204_L3.6mm_D1.6mm_P7.62mm_Horizontal -> Resistor_THT:R_Axial_DIN0207_L6.3mm_D2.5mm_P2.54mm_Vertical
- R12: value 15k -> 330; footprint Resistor_THT:R_Axial_DIN0204_L3.6mm_D1.6mm_P7.62mm_Horizontal -> Resistor_THT:R_Axial_DIN0207_L6.3mm_D2.5mm_P2.54mm_Vertical
- R16, R17: value 0.22 -> 0.33
- R18: value 1.5k -> 330
- R19: value 1.5k -> 1k
- R20: footprint Resistor_THT:R_Axial_DIN0414_L11.9mm_D4.5mm_P15.24mm_Horizontal -> Resistor_THT:R_Axial_DIN0516_L15.5mm_D5.0mm_P5.08mm_Vertical
- R3, R4, R5: value 1k -> 470
- R6: value 10k -> 4.7k
- R7: value 1k -> 2.2k
- R9: value 22k -> 47k
- RV1: value 10k -> 300
- moved R19 81.4 mm to (221.6, 44.5), turned to -90 degrees
- moved Q11 67.8 mm to (203.8, 73.0), turned to 0 degrees
- moved Q12 62.6 mm to (209.6, 85.9), turned to 0 degrees
- moved C1 62.1 mm to (201.7, 50.8)
- moved R2 60.1 mm to (196.2, 45.1), turned to 90 degrees
- moved R1 55.4 mm to (202.6, 45.1), turned to 90 degrees
- moved Q8 48.5 mm to (219.1, 84.1)
- moved Q3 48.0 mm to (213.9, 33.0), turned to -90 degrees
- moved C2 47.7 mm to (195.6, 50.2), turned to -90 degrees
- moved R14 44.3 mm to (214.0, 92.7)
- moved Q1 43.7 mm to (214.0, 43.2), turned to -90 degrees
- moved D5 43.6 mm to (255.9, 52.7), turned to 90 degrees
- moved R6 42.8 mm to (198.8, 70.5), turned to -90 degrees
- moved Q10 42.4 mm to (272.4, 84.7)
- moved J3 41.0 mm to (198.1, 59.8)
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Connections:
- net /INPUT renamed Net-(J3-Pin_2)
- C13 pad 1: GND -> PWRGND
- C14 pad 2: GND -> PWRGND
- C15 pad 2: GND -> PWRGND
- C16 pad 1: GND -> PWRGND
- C2 pad 1: Net-(Q1-B) -> Net-(Q2-B)
- C3 pad 1: Net-(Q13-E) -> Net-(D11-K)
- C4 pad 1: Net-(Q2-B) -> Net-(Q1-B)
- C5 pad 1: Net-(Q1-C) -> Net-(Q16-B)
- C5 pad 2: Net-(D6-A) -> Net-(D6-K)
- C6 pad 1: Net-(D6-A) -> Net-(D6-K)
- C6 pad 2: Net-(D3-K) -> Net-(D4-K)
- D10 pad 1: GND -> PWRGND
- D4 pad 2: Net-(D4-A) -> Net-(D11-A)
- D5 pad 1: B- -> Net-(D11-K)
- D5 pad 2: Net-(D4-K) -> Net-(D5-A)
- D6 pad 2: Net-(D6-A) -> Net-(D5-A)
- D7 pad 2: GND -> PWRGND
- J1 pad 2: GND -> PWRGND
- Q1 pad 1: Net-(Q1-C) -> Net-(Q1-E)
- Q1 pad 3: Net-(Q1-E) -> /LTP COM
- Q10 pad 1: Net-(Q10-B) -> Net-(Q10-G)
- Q10 pad 2: B+ -> B-
- Q10 pad 3: Net-(D8-A) -> Net-(D9-K)
- Q11 pad 1: Net-(Q11-E) -> B-
- Q11 pad 2: B- -> Net-(Q11-B)
- Q11 pad 3: Net-(D3-K) -> Net-(Q11-C)
- Q12 pad 1: Net-(Q11-E) -> B-
- Q12 pad 2: B- -> Net-(Q12-B)
- Q12 pad 3: Net-(D9-K) -> Net-(Q12-C)
- Q2 pad 1: /LTP COM -> Net-(Q2-E)
- Q2 pad 3: Net-(Q2-E) -> Net-(Q16-B)
- Q3 pad 1: Net-(Q1-C) -> Net-(Q3-E)
- Q3 pad 3: Net-(Q3-E) -> /LTP COM
- Q4 pad 1: /LTP COM -> Net-(Q4-E)
- Q4 pad 3: Net-(Q4-E) -> Net-(Q16-B)
- Q6 pad 2: Net-(D6-A) -> Net-(D6-K)
- Q6 pad 3: Net-(Q1-C) -> Net-(Q16-E)
- Q7 pad 1: Net-(D3-K) -> Net-(D4-K)
- Q7 pad 2: Net-(D6-A) -> Net-(D6-K)
- Q8 pad 1: Net-(Q8-E) -> Net-(Q12-B)
- Q8 pad 2: Net-(D3-K) -> Net-(D4-K)
- Q8 pad 3: Net-(D4-A) -> Net-(Q12-C)
- Q9 pad 1: Net-(Q10-B) -> Net-(Q9-G)
- Q9 pad 3: Net-(D6-A) -> Net-(D8-A)
- R1 pad 2: Net-(Q1-B) -> Net-(Q2-B)
- R11 pad 1: Net-(D6-A) -> Net-(D6-K)
- R12 pad 2: Net-(D3-K) -> Net-(D4-K)
- R13 pad 1: Net-(D4-A) -> Net-(Q12-C)
- R14 pad 1: Net-(Q8-E) -> Net-(Q12-B)
- R16 pad 2: Net-(Q13-E) -> Net-(D11-K)
- R17 pad 1: Net-(Q13-E) -> Net-(D11-K)
- R18 pad 1: Net-(Q10-B) -> Net-(D4-K)
- R18 pad 2: Net-(D8-A) -> Net-(Q10-G)
- R19 pad 1: Net-(D9-K) -> B+
- R19 pad 2: Net-(Q11-E) -> Net-(Q16-E)
- R2 pad 1: Net-(Q1-B) -> Net-(Q2-B)
- R20 pad 1: Net-(C3-Pad2) -> PWRGND
- R20 pad 2: GND -> Net-(C3-Pad2)
- R21 pad 1: Net-(Q13-E) -> Net-(D11-K)
- R3 pad 2: Net-(Q3-E) -> Net-(Q4-E)
- R4 pad 2: Net-(Q4-E) -> Net-(Q3-E)
- R5 pad 1: Net-(Q5-E) -> Net-(Q11-B)
- R6 pad 1: Net-(D1-A) -> Net-(Q11-C)
- R9 pad 1: Net-(Q2-B) -> Net-(Q1-B)
- R9 pad 2: Net-(Q13-E) -> Net-(D11-K)
Routing:
- net B-: track 20.5 -> 158.6 mm
- net PWRGND: track 0.00 -> 123.9 mm
- net GND: track 29.8 -> 145.6 mm
- net B+: track 0.00 -> 109.3 mm
- net Net-(D6-A): track 100.5 -> 0.00 mm
- net Net-(D11-K): track 0.00 -> 98.9 mm
- net Net-(Q13-E): track 95.7 -> 0.00 mm
- net Net-(D4-K): track 4.70 -> 85.4 mm
- net Net-(D3-K): track 74.3 -> 0.00 mm
- net Net-(Q16-B): track 0.00 -> 49.4 mm, vias 0 -> 1
- net Net-(D9-K): track 66.6 -> 17.9 mm
- net Net-(D8-A): track 79.4 -> 31.4 mm
- net Net-(Q1-C): track 47.6 -> 0.00 mm, vias 2 -> 0
- net Net-(D3-A): track 40.4 -> 0.00 mm
- net Net-(D4-A): track 34.0 -> 0.00 mm
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- removed copper zone on B.Cu, net /LTP COM
- removed copper zone on B.Cu, net B+
- removed copper zone on B.Cu, net B-
- removed copper zone on B.Cu, net GND
Other:
- board size 87.4 x 101.9 mm -> 84.5 x 82.5 mm
- board text added: "Designed By Pontus Rydin"
- board text added: "https://github.com/prydin/classab-amp-mosfet"
- board text removed: "Designed by Pontus Rydin. https://github.com/prydin/classab-amp"
- board text removed: "GND"
- board text removed: "V+"
- board text removed: "V-"

Commit message: Production candidate
Parts:
- C1, C6: footprint Capacitor_THT:CP_Radial_D4.0mm_P1.50mm -> Capacitor_THT:CP_Radial_D4.0mm_P2.00mm
- moved Q8 12.0 mm to (224.4, 94.9)
- moved Q12 4.68 mm to (214.1, 86.9)
- moved R21 1.30 mm to (247.7, 83.6)
- moved R2 0.54 mm to (195.8, 44.7)
- moved R1 0.35 mm to (202.6, 44.7)
Connections:
- R2 pad 1: Net-(Q2-B) -> GND
- R2 pad 2: GND -> Net-(Q2-B)
Routing:
- net B-: track 158.6 -> 147.6 mm
- net Net-(Q12-C): track 9.66 -> 15.9 mm
- net Net-(Q12-B): track 17.5 -> 20.8 mm
- net GND: track 145.6 -> 142.4 mm
- net Net-(Q2-B): track 18.7 -> 21.7 mm
- net Net-(D11-K): track 98.9 -> 96.3 mm
- net /SPEAKER: track 12.3 -> 13.7 mm
- net Net-(D4-K): track 85.4 -> 86.2 mm

Commit message: Production candidate
Parts:
- moved D9 2.32 mm to (258.1, 103.1)
Routing:
- net B-: track 147.6 -> 137.2 mm
- net Net-(D9-K): track 17.9 -> 18.9 mm
Other:
- board text added: "B+"
- board text added: "B-"
- board text added: "GND"
- board text added: "IN"
Changed lines of the file:
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@@
 		(at 263.525 104.775)
 		(property "Reference" "J2"
-			(at 0 1.805 0)
+			(at -6.477 5.08 0)
 			(unlocked yes)
 			(layer "F.SilkS")
@@
 		(at 262.89 30.48)
 		(property "Reference" "J4"
-			(at 0 1.27 0)
+			(at 6.096 7.112 0)
 			(unlocked yes)
 			(layer "F.SilkS")
@@
 	(footprint "Diode_THT:D_DO-41_SOD81_P10.16mm_Horizontal"
 		(layer "F.Cu")
-		(at 260.35 103.505)
+		(at 258.064 103.124)
 		(descr "Diode, DO-41_SOD81 series, Axial, Horizontal, pin pitch=10.16mm, , length*diameter=5.2*2.7mm^2, , http://www.diodes.com/_files/packages/DO-41%20(Plastic).pdf")
 		(tags "Diode DO-41_SOD81 series Axial Horizontal pin pitch 10.16mm  length 5.2mm diameter 2.7mm")
@@
 		(tags "Resistor Axial_DIN0207 series Axial Vertical pin pitch 2.54mm 0.25W = 1/4W length 6.3mm diameter 2.5mm")
 		(property "Reference" "R2"
-			(at 4.572 0 360)
+			(at 4.572 0 0)
 			(layer "F.SilkS")
 			(effects
@@
 		(layer "Edge.Cuts")
 	)
+	(gr_text "B+"
+		(at 262.89 33.02 0)
+		(layer "F.SilkS")
+		(effects
+			(font
+				(size 1.5 1.5)
+				(thickness 0.1)
+			)
+			(justify bottom)
+		)
+	)
 	(gr_text "https://github.com/prydin/classab-amp-mosfet"
 		(at 201.93 111.125 0)
@@
 		)
 	)
+	(gr_text "IN"
+		(at 198.12 66.802 0)
+		(layer "F.SilkS")
+		(effects
+			(font
+				(size 1 1)
+				(thickness 0.1)
+			)
+			(justify bottom)
+		)
+	)
+	(gr_text "B-"
+		(at 263.525 107.315 0)
+		(layer "F.SilkS")
+		(effects
+			(font
+				(size 1.5 1.5)
+				(thickness 0.1)
+			)
+			(justify bottom)
+		)
+	)
+	(gr_text "GND"
+		(at 198.02 57.665 0)
+		(layer "F.SilkS")
+		(effects
+			(font
+				(size 1 1)
+				(thickness 0.1)
+			)
+			(justify bottom)
+		)
+	)
+	(gr_text "GND"
+		(at 223.52 85.725 90)
+		(layer "F.SilkS")
+		(effects
+			(font
+				(size 1.5 1.5)
+				(thickness 0.1)
+			)
+			(justify bottom)
+		)
+	)
 	(segment
 		(start 199.817056 63.325)
@@
 	)
 	(segment
+		(start 260.35 99.06)
+		(end 260.35 100.838)
+		(width 5)
+		(layer "F.Cu")
+		(net 15)
+	)
+	(segment
 		(start 263.79 95.62)
 		(end 260.35 99.06)
@@
 	)
 	(segment
-		(start 260.35 103.505)
-		(end 260.35 99.06)
-		(width 2)
+		(start 258.064 103.124)
+		(end 258.064 103.505)
+		(width 5)
 		(layer "F.Cu")
 		(net 15)
@@
 	)
 	(segment
+		(start 260.35 100.838)
+		(end 258.064 103.124)
+		(width 5)
+		(layer "F.Cu")
+		(net 15)
+	)
+	(segment
 		(start 202.565 45.085)
 		(end 203.835 46.355)
@@
 	)
 	(segment
-		(start 270.51 103.505)
-		(end 270.51 101.115)
-		(width 2)
+		(start 266.065 109.855)
+		(end 266.065 103.124)
+		(width 5)
 		(layer "B.Cu")
 		(net 22)
@@
 	)
 	(segment
+		(start 266.065 103.124)
+		(end 266.065 96.67)
+		(width 5)
+		(layer "B.Cu")
+		(net 22)
+	)
+	(segment
 		(start 266.065 96.67)
 		(end 263.365 93.97)
@@
 	)
 	(segment
+		(start 268.224 103.124)
+		(end 266.065 103.124)
+		(width 5)
+		(layer "B.Cu")
+		(net 22)
+	)
+	(segment
 		(start 238.552056 99.695)
 		(end 240.747056 101.89)
@@
 	)
 	(segment
-		(start 270.51 101.115)
-		(end 263.365 93.97)
-		(width 2)
-		(layer "B.Cu")
-		(net 22)
-	)
-	(segment
 		(start 263.365 93.97)
 		(end 267.165 90.17)
@@
 		(width 5)
 		(layer "B.Cu")
-		(net 22)
-	)
-	(segment
-		(start 266.065 109.855)
-		(end 266.065 96.67)
-		(width 5)
-		(layer "B.Cu")

Commit message: Public release candidate
Parts:
- added R22: 100, Resistor_THT:R_Axial_DIN0204_L3.6mm_D1.6mm_P7.62mm_Horizontal, F.Cu at (195.6, 70.6)
- R1: value 2.2k -> 150
- R7: value 2.2k -> 1k
- R9: value 47k -> 22k
- moved D4 7.38 mm to (255.5, 90.4), turned to -90 degrees
- moved Q8 3.94 mm to (220.5, 94.9)
- moved R13 2.54 mm to (216.5, 92.7)
- moved R14 2.54 mm to (211.5, 92.7)
- moved J5 1.52 mm to (219.5, 85.7)
- moved R6 0.65 mm to (199.4, 70.6)
Connections:
- C2 pad 2: GND -> PWRGND
- C7 pad 1: GND -> PWRGND
- J3 pad 1: GND -> GNDS
- Q16 pad 3: GND -> PWRGND
- R13 pad 2: GND -> PWRGND
- R15 pad 2: GND -> PWRGND
- R2 pad 1: GND -> PWRGND
- R6 pad 2: GND -> PWRGND
- R7 pad 1: GND -> PWRGND
Routing:
- net PWRGND: track 123.9 -> 357.0 mm
- net GND: track 142.4 -> 0.00 mm
- net GNDS: track 0.00 -> 11.8 mm
- net Net-(D4-K): track 86.2 -> 75.3 mm
- net Net-(D11-A): track 9.99 -> 5.44 mm
- net B-: track 137.2 -> 141.2 mm
- net Net-(Q12-C): track 15.9 -> 15.1 mm
- net Net-(Q11-C): track 24.0 -> 23.5 mm

Commit message: Update classab-amp.kicad_pcb
Parts:
- removed RV2: 300, footprints:TRIM_T93YA103KT20
- added D1: 1N4148, Diode_THT:D_DO-35_SOD27_P7.62mm_Horizontal, F.Cu at (220.5, 69.6)
- added R23: 100, Resistor_THT:R_Axial_DIN0207_L6.3mm_D2.5mm_P2.54mm_Vertical, F.Cu at (213.4, 55.9)
- added R24: 100, Resistor_THT:R_Axial_DIN0207_L6.3mm_D2.5mm_P2.54mm_Vertical, F.Cu at (208.8, 53.8)
- C1: value 33u -> 4.7u
- moved J3 0.88 mm to (198.1, 60.7)
Routing:
- net PWRGND: track 357.0 -> 347.1 mm
- net Net-(D1-K): track 49.4 -> 54.6 mm
- net Net-(D1-A): track 73.2 -> 77.4 mm
- net Net-(Q15-C): track 13.1 -> 13.8 mm
- net Net-(Q2-E): track 5.40 -> 5.96 mm

Commit message: Pre re-layout
Parts:
- removed ?: , 
- removed D1: 1N4148, Diode_THT:D_DO-35_SOD27_P7.62mm_Horizontal
- removed D11: 1N5919, Diode_THT:D_DO-41_SOD81_P10.16mm_Horizontal
- removed D8, D9: 1N4004, Diode_THT:D_DO-41_SOD81_P10.16mm_Horizontal
- removed R16, R17: 0.33, Resistor_THT:R_Axial_DIN0414_L11.9mm_D4.5mm_P15.24mm_Horizontal
- removed R21: 10, Resistor_THT:R_Axial_DIN0414_L11.9mm_D4.5mm_P15.24mm_Horizontal
- removed the REF** at (196.8, 34.3)
- removed the REF** at (273.7, 34.3)
- added C10: 68p, Capacitor_THT:C_Rect_L7.2mm_W3.0mm_P5.00mm_FKS2_FKP2_MKS2_MKP2, F.Cu at (250.2, 117.3)
- added C8: 220n, Capacitor_THT:C_Rect_L7.2mm_W3.0mm_P5.00mm_FKS2_FKP2_MKS2_MKP2, F.Cu at (260.6, 98.8)
- added C9: 68p, Capacitor_THT:C_Rect_L7.2mm_W3.0mm_P5.00mm_FKS2_FKP2_MKS2_MKP2, F.Cu at (250.2, 75.9)
- added D2: 1N4148, Diode_THT:D_DO-35_SOD27_P7.62mm_Horizontal, F.Cu at (216.9, 125.7)
- added D3: 1N5919, Diode_THT:D_DO-41_SOD81_P10.16mm_Horizontal, F.Cu at (255.3, 62.0)
- added J6: ~, footprints:Spade Connector, F.Cu at (215.1, 97.3)
- added Q13: BD139, Package_TO_SOT_THT:TO-126-3_Vertical, F.Cu at (271.0, 81.9)
- added Q14: BD140, Package_TO_SOT_THT:TO-126-3_Vertical, F.Cu at (271.3, 105.2)
- added Q5: 2N5551, Package_TO_SOT_THT:TO-92_Wide, F.Cu at (223.5, 142.5)
- added R25: 100, Resistor_THT:R_Axial_DIN0207_L6.3mm_D2.5mm_P2.54mm_Vertical, F.Cu at (223.5, 129.8)
- added REF**: MountingHole_3.2mm_M3, MountingHole:MountingHole_3.2mm_M3, F.Cu at (271.8, 36.1)
- added REF**: MountingHole_3.2mm_M3, MountingHole:MountingHole_3.2mm_M3, F.Cu at (216.4, 36.1)
- added REF**: MountingHole_3.2mm_M3, MountingHole:MountingHole_3.2mm_M3, F.Cu at (216.4, 154.4)
- C5: value 100p -> 33p
- D5: value 1N4148 -> 1N5919; footprint Diode_THT:D_DO-35_SOD27_P7.62mm_Horizontal -> Diode_THT:D_DO-41_SOD81_P10.16mm_Horizontal
- D6: value 1N5919 -> 1N4148; footprint Diode_THT:D_DO-41_SOD81_P10.16mm_Horizontal -> Diode_THT:D_DO-35_SOD27_P7.62mm_Horizontal
- J1: value SPEAKER -> ~; footprint TerminalBlock_Phoenix:TerminalBlock_Phoenix_MKDS-1,5-2_1x02_P5.00mm_Horizontal -> footprints:Spade Connector
- Q1, Q2: value 2N5551 -> 2N5401
- Q6: value BD140 -> 2N5401; footprint Package_TO_SOT_THT:TO-126-3_Vertical -> Package_TO_SOT_THT:TO-92_Wide
- Q8: value BD139 -> 2N5551; footprint Package_TO_SOT_THT:TO-126-3_Vertical -> Package_TO_SOT_THT:TO-92_Wide
- R1, R2: footprint Resistor_THT:R_Axial_DIN0207_L6.3mm_D2.5mm_P2.54mm_Vertical -> Resistor_THT:R_Axial_DIN0204_L3.6mm_D1.6mm_P7.62mm_Horizontal
- R10: value 100 -> 47
- R11: value 4.7k -> 10k
- R12: value 330 -> 680
- R13: value 10k -> 1k
- R14: value 100 -> 10k
- R18, R8: value 330 -> 47
- R19: value 1k -> 10k
- R20: footprint Resistor_THT:R_Axial_DIN0516_L15.5mm_D5.0mm_P5.08mm_Vertical -> Resistor_THT:R_Axial_DIN0414_L11.9mm_D4.5mm_P15.24mm_Horizontal
- R23: value 100 -> 680; footprint Resistor_THT:R_Axial_DIN0207_L6.3mm_D2.5mm_P2.54mm_Vertical -> Resistor_THT:R_Axial_DIN0204_L3.6mm_D1.6mm_P7.62mm_Horizontal
- R4: value 470 -> 1k
- R6: value 4.7k -> 22
- moved R3 113.6 mm to (229.6, 147.6), turned to 0 degrees
- moved Q1 96.2 mm to (219.4, 139.2), turned to 90 degrees
- moved Q2 87.0 mm to (223.5, 134.1), turned to -90 degrees
- moved Q4 77.5 mm to (219.2, 115.1)
- moved Q3 77.5 mm to (223.3, 110.0)
- moved R5 76.8 mm to (229.6, 151.9), turned to 0 degrees
- moved R24 76.5 mm to (217.6, 129.8), turned to 0 degrees
- moved Q11 76.2 mm to (219.5, 147.6), turned to 90 degrees
- moved Q15 75.4 mm to (236.0, 133.6)
- moved R6 72.0 mm to (250.4, 121.4)
- moved D6 69.2 mm to (265.7, 122.7), turned to 180 degrees
- moved R23 68.4 mm to (265.4, 100.3)
- moved C7 66.8 mm to (236.4, 38.9), turned to 180 degrees
- moved R7 62.3 mm to (230.6, 119.1), turned to 90 degrees
- moved R15 61.9 mm to (226.6, 47.0), turned to 0 degrees
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Connections:
- C2 pad 1: Net-(Q2-B) -> Net-(Q1-B)
- C3 pad 1: Net-(D11-K) -> /SPEAKER
- C4 pad 1: Net-(Q1-B) -> Net-(D2-K)
- C4 pad 2: Net-(C4-Pad2) -> PWRGND
- C5 pad 1: Net-(D1-K) -> Net-(Q1-C)
- C5 pad 2: Net-(D1-A) -> Net-(Q14-B)
- C6 pad 1: Net-(D1-A) -> Net-(Q13-B)
- C6 pad 2: Net-(D4-K) -> Net-(Q14-B)
- D4 pad 1: Net-(D4-K) -> /SPEAKER
- D5 pad 1: Net-(D11-K) -> /SPEAKER
- D6 pad 1: Net-(D1-A) -> Net-(D6-K)
- J1 pad 2: PWRGND -> /SPEAKER
- Q1 pad 3: /LTP COM -> Net-(Q1-C)
- Q10 pad 1: Net-(Q10-G) -> Net-(D6-K)
- Q10 pad 3: Net-(D9-K) -> /SPEAKER
- Q11 pad 1: B- -> Net-(Q11-E)
- Q11 pad 3: Net-(Q11-C) -> Net-(Q1-C)
- Q12 pad 1: B- -> Net-(Q12-E)
- Q12 pad 2: Net-(Q12-B) -> Net-(Q1-C)
- Q12 pad 3: Net-(Q12-C) -> PWRGND
- Q15 pad 1: Net-(Q11-B) -> B-
- Q15 pad 2: Net-(Q11-C) -> Net-(Q15-B)
- Q15 pad 3: Net-(Q15-C) -> Net-(Q1-C)
- Q16 pad 2: Net-(D1-K) -> Net-(Q16-B)
- Q16 pad 3: PWRGND -> Net-(Q13-B)
- Q2 pad 1: Net-(Q2-E) -> /LTP COM
- Q2 pad 3: Net-(D1-K) -> Net-(Q11-B)
- Q3 pad 2: /LTP COM -> Net-(Q3-B)
- Q3 pad 3: /LTP COM -> Net-(Q3-C)
- Q4 pad 1: Net-(Q4-E) -> B+
- Q4 pad 2: /LTP COM -> Net-(Q3-E)
- Q4 pad 3: Net-(D1-K) -> Net-(Q3-B)
- Q6 pad 1: Net-(Q6-E) -> B+
- Q6 pad 2: Net-(D1-A) -> Net-(Q16-E)
- Q6 pad 3: Net-(Q16-E) -> Net-(Q16-B)
- Q7 pad 1: Net-(D4-K) -> Net-(Q14-B)
- Q7 pad 2: Net-(D1-A) -> Net-(Q13-B)
- Q8 pad 1: Net-(Q12-B) -> Net-(Q15-B)
- Q8 pad 2: Net-(D4-K) -> Net-(Q12-E)
- Q8 pad 3: Net-(Q12-C) -> Net-(Q14-B)
- Q9 pad 3: Net-(D8-A) -> /SPEAKER
- R1 pad 2: Net-(Q2-B) -> Net-(Q1-B)
- R10 pad 2: Net-(Q6-E) -> Net-(Q16-E)
- R11 pad 1: Net-(D1-A) -> Net-(Q13-B)
- R12 pad 2: Net-(D4-K) -> Net-(Q14-B)
- R13 pad 1: Net-(Q12-C) -> Net-(Q12-E)
- R13 pad 2: PWRGND -> B-
- R14 pad 1: Net-(Q12-B) -> Net-(Q16-B)
- R14 pad 2: B- -> PWRGND
- R18 pad 1: Net-(D4-K) -> Net-(Q14-E)
- R18 pad 2: Net-(Q10-G) -> Net-(D6-K)
- R19 pad 1: B+ -> Net-(Q3-B)
- R19 pad 2: Net-(Q16-E) -> PWRGND
- R2 pad 2: Net-(Q2-B) -> Net-(Q1-B)
- R23 pad 1: Net-(Q15-C) -> Net-(Q13-E)
- R23 pad 2: Net-(Q1-E) -> Net-(Q14-E)
- R24 pad 1: Net-(Q2-E) -> Net-(Q1-E)
- R24 pad 2: Net-(Q15-C) -> Net-(Q3-C)
- R3 pad 1: B+ -> Net-(Q11-E)
- R3 pad 2: Net-(Q4-E) -> B-
- R5 pad 1: Net-(Q11-B) -> Net-(Q5-E)
- R6 pad 1: Net-(Q11-C) -> Net-(Q15-B)
- R6 pad 2: PWRGND -> B-
- R7 pad 1: PWRGND -> Net-(D2-K)
- R7 pad 2: Net-(C4-Pad2) -> Net-(Q2-B)
- R8 pad 1: Net-(D1-A) -> Net-(Q13-E)
- R9 pad 1: Net-(Q1-B) -> Net-(Q2-B)
- R9 pad 2: Net-(D11-K) -> /SPEAKER
Routing:
- net Net-(Q14-B): track 0.00 -> 96.6 mm
- net Net-(D11-K): track 96.3 -> 0.00 mm
- net /SPEAKER: track 13.7 -> 100.5 mm
- net Net-(D1-A): track 77.4 -> 0.00 mm
- net Net-(D4-K): track 75.3 -> 0.00 mm
- net Net-(Q13-E): track 0.00 -> 70.6 mm
- net Net-(Q13-B): track 0.00 -> 69.3 mm
- net PWRGND: track 347.1 -> 290.6 mm
- net B+: track 109.3 -> 165.6 mm
- net Net-(D1-K): track 54.6 -> 0.00 mm, vias 1 -> 0
- net Net-(Q1-C): track 0.00 -> 50.7 mm
- net Net-(Q1-B): track 31.0 -> 79.4 mm
- net Net-(Q14-E): track 0.00 -> 45.3 mm
- net Net-(Q15-B): track 0.00 -> 36.9 mm
- net Net-(D8-A): track 31.4 -> 0.00 mm
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Other:
- board size 84.5 x 82.5 mm -> 62.6 x 125.7 mm
- board text added: "SPK"
- board text removed: "Designed By Pontus Rydin"
- board text removed: "IN"
- board text removed: "https://github.com/prydin/classab-amp-mosfet"

Commit message: WIP
Parts:
- Q16: value 2N5401 -> BD140; footprint Package_TO_SOT_THT:TO-92_Wide -> Package_TO_SOT_THT:TO-126-3_Vertical
- Q8: value 2N5551 -> BD139; footprint Package_TO_SOT_THT:TO-92_Wide -> Package_TO_SOT_THT:TO-126-3_Vertical
- moved J6 19.7 mm to (234.8, 97.5)
- moved J5 18.4 mm to (240.9, 97.5)
- moved Q2 15.2 mm to (223.8, 118.9)
- moved Q1 15.2 mm to (219.5, 124.0)
- moved R24 15.0 mm to (217.4, 114.8)
- moved R25 15.0 mm to (223.7, 114.8)
- moved Q4 11.2 mm to (224.0, 104.9), turned to -90 degrees
- moved D2 11.2 mm to (216.9, 136.9)
- moved C4 10.9 mm to (221.6, 133.1)
- moved C7 10.5 mm to (231.9, 48.3)
- moved R19 10.3 mm to (216.7, 100.6), turned to 90 degrees
- moved R11 10.3 mm to (232.9, 90.1)
- moved RV1 10.2 mm to (226.8, 97.5)
- moved R12 10.2 mm to (233.2, 103.7)
- moved C6 10.2 mm to (232.5, 97.3)
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Connections:
- Q16 pad 2: Net-(Q16-B) -> Net-(Q13-B)
- Q16 pad 3: Net-(Q13-B) -> Net-(Q16-B)
- Q8 pad 2: Net-(Q12-E) -> Net-(Q14-B)
- Q8 pad 3: Net-(Q14-B) -> Net-(Q12-E)
Routing:
- net PWRGND: track 290.6 -> 334.9 mm
- net Net-(Q11-B): track 18.1 -> 51.6 mm
- net Net-(Q1-C): track 50.7 -> 72.6 mm
- net Net-(Q1-B): track 79.4 -> 63.8 mm
- net Net-(Q2-B): track 48.1 -> 32.8 mm
- net Net-(Q13-B): track 69.3 -> 81.6 mm
- net B+: track 165.6 -> 153.7 mm
- net Net-(Q3-E): track 30.4 -> 18.6 mm
- net Net-(Q7-B): track 43.7 -> 54.0 mm
- net Net-(D2-K): track 16.5 -> 23.6 mm
- net Net-(Q3-C): track 20.0 -> 14.6 mm
- net CHASSIS: track 25.3 -> 20.1 mm
- net Net-(Q3-B): track 14.8 -> 18.6 mm
- net Net-(Q16-B): track 23.6 -> 20.4 mm
- net B-: track 123.2 -> 121.6 mm
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Other:
- board text added: "R19"
- board text added: "R7"

Commit message: WIP
Parts:
- added C11: 4.7u, Capacitor_THT:CP_Radial_D4.0mm_P2.00mm, F.Cu at (236.9, 52.8)
- added D1: 1N4148, Diode_THT:D_DO-35_SOD27_P5.08mm_Vertical_KathodeUp, F.Cu at (229.7, 108.5)
- added D8: 1N4148, Diode_THT:D_DO-35_SOD27_P7.62mm_Horizontal, F.Cu at (224.3, 131.3)
- added D9: 1N4148, Diode_THT:D_DO-35_SOD27_P7.62mm_Horizontal, F.Cu at (216.7, 127.8)
- added R16: 4.7k, Resistor_THT:R_Axial_DIN0204_L3.6mm_D1.6mm_P7.62mm_Horizontal, F.Cu at (232.2, 58.2)
- C7: value 10n -> 4.7u; footprint Capacitor_THT:C_Rect_L7.2mm_W3.0mm_P5.00mm_FKS2_FKP2_MKS2_MKP2 -> Capacitor_THT:CP_Radial_D4.0mm_P2.00mm
- R14, R19: value 10k -> 4.7k
- R15: value 220 -> 4.7k; footprint Resistor_THT:R_Axial_DIN0414_L11.9mm_D4.5mm_P15.24mm_Horizontal -> Resistor_THT:R_Axial_DIN0204_L3.6mm_D1.6mm_P7.62mm_Horizontal
- R20: footprint Resistor_THT:R_Axial_DIN0414_L11.9mm_D4.5mm_P15.24mm_Horizontal -> Resistor_THT:R_Axial_DIN0414_L11.9mm_D4.5mm_P5.08mm_Vertical
- moved R15 46.1 mm to (216.4, 88.4)
- moved C7 33.5 mm to (222.0, 80.3)
- moved R22 17.2 mm to (223.3, 69.6), turned to 0 degrees
- moved R14 12.4 mm to (240.8, 65.3), turned to 90 degrees
- moved R20 11.4 mm to (240.0, 82.8)
- moved C4 8.76 mm to (226.6, 140.3), turned to 90 degrees
- moved R6 8.52 mm to (254.3, 113.8)
- moved D2 4.83 mm to (217.2, 141.7)
- moved Q5 2.06 mm to (223.8, 144.6)
- moved R5 2.06 mm to (229.6, 153.9)
- moved Q11 2.06 mm to (219.5, 149.6)
- moved R3 2.06 mm to (229.6, 149.6)
- moved Q6 1.78 mm to (233.9, 70.6)
- moved Q8 1.14 mm to (253.2, 109.9)
- moved R18 0.25 mm to (264.9, 116.8)
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Connections:
- C7 pad 1: PWRGND -> B+
- C7 pad 2: CHASSIS -> Net-(C7-Pad2)
- R14 pad 2: PWRGND -> Net-(C11-Pad2)
- R15 pad 1: CHASSIS -> Net-(C7-Pad2)
- R19 pad 2: PWRGND -> Net-(C7-Pad2)
- REF** pad : CHASSIS -> (no net)
Routing:
- net CHASSIS: track 20.1 -> 0.00 mm
- net Net-(C11-Pad2): track 0.00 -> 15.0 mm
- net Net-(D2-K): track 23.6 -> 38.2 mm
- net Net-(C7-Pad2): track 0.00 -> 14.5 mm
- net Net-(D1-A): track 32.8 -> 45.8 mm
- net Net-(D8-A): track 63.8 -> 75.0 mm
- net Net-(Q1-C): track 72.6 -> 83.0 mm
- net /LTP COM: track 5.11 -> 12.9 mm
- net B+: track 153.7 -> 161.4 mm
- net GNDS: track 17.9 -> 11.3 mm
- net PWRGND: track 334.9 -> 339.2 mm
- net Net-(Q11-B): track 51.6 -> 48.0 mm
- net Net-(Q15-B): track 35.6 -> 37.6 mm
- net Net-(Q16-E): track 20.7 -> 22.4 mm
- net Net-(C3-Pad2): track 8.27 -> 6.99 mm
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Other:
- board text added: "IN"
- board text added: "The Bog Standard 50W"
